File: hardware/capteur.kicad_pcb (KiCad board)
At the start: 2 copper layers, 69.8 x 60 mm, 32 parts, among them P1 CONN_5, P2 CONN_2, P3 CONN_6, P4 CONN_4, P5 CONN_4, U1 PIC18F2XK80, U2 STEVAL-MKI108V2, U3 MCP2562, U4 UA78M33, U5 UA78M05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

Commit message: Convert to kicad 6.x
Connections:
- net /~MCLR renamed /~{MCLR}
Other:
- net class Default removed
