File: hardware/clk-command.sch (KiCad schematic (older format))
At the start: 10 parts, among them P1 CONN_1, P2 CONN_1, P3 CONN_1, P4 CONN_1, U1 74HC14, X1 CRYSTAL

Commit message: Convert to kicad 6.x
Parts:
- C1, C2, C3: symbol C -> clk-command-rescue:C
- P1, P2, P3, P4: symbol CONN_1 -> clk-command-rescue:CONN_1
- R1: symbol R -> clk-command-rescue:R
- U1: symbol 74HC14 -> clk-command-rescue:74HC14
- X1: symbol CRYSTAL -> clk-command-rescue:CRYSTAL
Connections:
- wire segments 19 -> 29
Changed lines of the file:
@@
-EESchema Schematic File Version 2
-LIBS:power
-LIBS:device
-LIBS:transistors
-LIBS:conn
-LIBS:linear
-LIBS:regul
-LIBS:74xx
-LIBS:cmos4000
-LIBS:adc-dac
-LIBS:memory
-LIBS:xilinx
-LIBS:special
-LIBS:microcontrollers
-LIBS:dsp
-LIBS:microchip
-LIBS:analog_switches
-LIBS:motorola
-LIBS:texas
-LIBS:intel
-LIBS:audio
-LIBS:interface
-LIBS:digital-audio
-LIBS:philips
-LIBS:display
-LIBS:cypress
-LIBS:siliconi
-LIBS:opto
-LIBS:atmel
-LIBS:contrib
-LIBS:valves
-LIBS:clk-command-cache
-EELAYER 27 0
+EESchema Schematic File Version 4
+EELAYER 30 0
 EELAYER END
 $Descr A4 11693 8268
@@
 $EndDescr
 $Comp
-L 74HC14 U1
+L clk-command-rescue:74HC14 U1
 U 2 1 532172E9
 P 4800 2550
@@
 $EndComp
 $Comp
-L 74HC14 U1
+L clk-command-rescue:74HC14 U1
 U 3 1 532172F8
 P 6050 2550
@@
 $EndComp
 $Comp
-L 74HC14 U1
+L clk-command-rescue:74HC14 U1
 U 1 1 53217307
 P 4850 3600
@@
 $EndComp
 $Comp
-L 74HC14 U1
+L clk-command-rescue:74HC14 U1
 U 4 1 53217316
 P 4850 4150
@@
 $EndComp
 $Comp
-L 74HC14 U1
+L clk-command-rescue:74HC14 U1
 U 5 1 53217325
 P 4850 4700
@@
 $EndComp
 $Comp
-L 74HC14 U1
+L clk-command-rescue:74HC14 U1
 U 6 1 53217334
 P 4850 5150
@@
 $EndComp
 $Comp
-L R R1
+L clk-command-rescue:R R1
 U 1 1 532173C4
 P 4800 2850
@@
 $EndComp
 $Comp
-L C C2
+L clk-command-rescue:C C2
 U 1 1 532173E4
 P 5250 1600
@@
 $EndComp
 $Comp
-L C C1
+L clk-command-rescue:C C1
 U 1 1 532173F1
 P 4350 1600
@@
 $EndComp
 $Comp
-L GND #PWR01
+L clk-command-rescue:GND #PWR01
 U 1 1 532173F9
 P 5250 1150
@@
 $EndComp
 $Comp
-L GND #PWR02
+L clk-command-rescue:GND #PWR02
 U 1 1 53217408
 P 4350 1150
@@
 $EndComp
 $Comp
-L CONN_1 P1
+L clk-command-rescue:CONN_1 P1
 U 1 1 53217453
 P 6400 900
@@
 $EndComp
 $Comp
-L CONN_1 P4
+L clk-command-rescue:CONN_1 P4
 U 1 1 53217466
 P 6800 2550
@@
 $EndComp
 $Comp
-L GND #PWR03
+L clk-command-rescue:GND #PWR03
 U 1 1 53217483
 P 5750 900
@@
 $EndComp
 $Comp
-L VCC #PWR04
+L clk-command-rescue:VCC #PWR04
 U 1 1 5321748B
 P 5800 1500
@@
 CLK
 $Comp
-L CRYSTAL X1
+L clk-command-rescue:CRYSTAL X1
 U 1 1 532174B3
 P 4800 1850
@@
 $EndComp
 $Comp
-L GND #PWR05
+L clk-command-rescue:GND #PWR05
 U 1 1 53217722
 P 6000 2800
@@
 $EndComp
 $Comp
-L VCC #PWR06
+L clk-command-rescue:VCC #PWR06
 U 1 1 5321773A
 P 6000 2300
@@
 NoConn ~ 5300 5150
 $Comp
-L PWR_FLAG #FLG07
+L clk-command-rescue:PWR_FLAG #FLG07
 U 1 1 53217776
 P 6250 800
@@
 $EndComp
 $Comp
-L PWR_FLAG #FLG08
+L clk-command-rescue:PWR_FLAG #FLG08
 U 1 1 53217785
 P 6250 1400
@@
 $EndComp
 $Comp
-L CONN_1 P3
+L clk-command-rescue:CONN_1 P3
 U 1 1 53221BE9
 P 6400 1500
@@
 $EndComp
 $Comp
-L GND #PWR09
+L clk-command-rescue:GND #PWR09
 U 1 1 532220B3
 P 4400 5300
@@
 $EndComp
 $Comp
-L CONN_1 P2
+L clk-command-rescue:CONN_1 P2
 U 1 1 53217460
 P 6400 1650
@@
 	4350 1150 4350 1400
 Wire Wire Line
-	4350 1800 4350 2850
+	4350 1800 4350 1850
 Wire Wire Line
 	4350 2850 4550 2850
@@
 	5250 2850 5050 2850
 Wire Wire Line
-	5250 1800 5250 2850
+	5250 1800 5250 1850
 Connection ~ 5250 2550
 Wire Wire Line
 	6500 2550 6650 2550
 Wire Wire Line
-	5750 900  6250 900
-Wire Wire Line
-	5800 1500 6250 1500
+	5750 900  5950 900
+Wire Wire Line
+	5800 1500 5950 1500
 Wire Wire Line
 	5100 1850 5250 1850
@@
 	6000 2300 6000 2450
 Wire Wire Line
-	6250 1400 6250 1650
+	6250 1400 6250 1500
 Connection ~ 6250 900
 Wire Wire Line
-	4400 3600 4400 5300
+	4400 3600 4400 4150
 Connection ~ 4400 4150
 Connection ~ 4400 4700
@@
 Connection ~ 6250 1500
 $Comp
-L C C3
+L clk-command-rescue:C C3
 U 1 1 53230A66
 P 5950 1200
@@
 	5950 1400 5950 1500
 Connection ~ 5950 1500
+Wire Wire Line
+	4350 2550 4350 2850
+Wire Wire Line
+	5250 2550 5250 2850
+Wire Wire Line
+	5250 1850 5250 2550
+Wire Wire Line
+	4350 1850 4350 2550
+Wire Wire Line
+	4400 4150 4400 4700
+Wire Wire Line
+	4400 4700 4400 5150
+Wire Wire Line
+	4400 5150 4400 5300
+Wire Wire Line
+	6250 1500 6250 1650
+Wire Wire Line
+	5950 900  6250 900
+Wire Wire Line
+	5950 1500 6250 1500
 $EndSCHEMATC
