File: hardware/clk-control-main.kicad_pcb (KiCad board)
At the start: 2 copper layers, 30.2 x 20.5 mm, 12 parts, among them P1 CONN_1, P2 CONN_1, P3 CONN_1, P4 CONN_1, P5 CONN_1, P6 CONN_1, U1 74HC14, X1 CRYSTAL

Commit message: Convert to kicad 6.x
Other:
- net class Default removed
