File: hardware/command.kicad_pcb (KiCad board)
At the start: 2 copper layers, 69.8 x 84.8 mm, 41 parts, among them K1 CONN_3, P1 CONN_6, P2 CONN_6, P3 CONN_2, P4 CONN_2, P5 CONN_4, P6 CONN_4, P7 CONN_2, Q1 FDD8780, U1 UA78M05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

Commit message: Convert to kicad 6.x
Connections:
- net /~MCLR renamed /~{MCLR}
Other:
- net class Default removed
