File: hardware/control-display.kicad_pcb (KiCad board)
At the start: 2 copper layers, 55 x 33 mm, 21 parts, among them IC1 LM3405, K1 CONN_3, P1 CONN_5, P2 CONN_2

Commit message: Convert to kicad 6.x
Other:
- net class Default removed
- net class larger removed
- net class power removed
