File: hardware/remote-control/remote-control.kicad_pcb (KiCad board)
At the start: 2 copper layers, 74 x 34 mm, 26 parts, among them J1 Conn_Coaxial, P1 CONN_6, P2 CONN_4, P3 CONN_4, U1 PIC18F2XK80, U2 MCP2562, U3 ZPT, U4 UA78M33, U5 UA78M05, Y1 10Mhz

Commit message: Convert to kicad 6.x
Connections:
- net /~MCLR renamed /~{MCLR}
Other:
- net class Default removed
- net class RF removed
