File: hardware/remote-control/remote-control.sch (KiCad schematic (older format))
At the start: 24 parts, among them J1 Conn_Coaxial, P1 CONN_6, P2 CONN_4, P3 CONN_4, U1 PIC18F2XK80, U2 MCP2562, U3 ZPT, U4 UA78M33, U5 UA78M05, Y1 10Mhz

Commit message: Convert to kicad 6.x
Parts:
- C1, C3: symbol remote-control-rescue:C_Small-Device -> remote-control-rescue:C_Small-Device-remote-control-rescue
- C2, C7, C8, C9: symbol remote-control-rescue:CP1-RESCUE-capteur-capteur-rescue -> remote-control-rescue:CP1-RESCUE-capteur-capteur-rescue-remote-control-rescue
- C4, C5: symbol remote-control-rescue:C-RESCUE-capteur-capteur-rescue -> remote-control-rescue:C-RESCUE-capteur-capteur-rescue-remote-control-rescue
- C6: symbol Device:C_Small -> remote-control-rescue:C_Small-Device-remote-control-rescue
- D1: symbol Device:LED -> remote-control-rescue:LED-Device
- D2: symbol Device:D_Schottky_Small -> remote-control-rescue:D_Schottky_Small-Device
- J1: symbol Connector:Conn_Coaxial -> remote-control-rescue:Conn_Coaxial-Connector
- P1: symbol remote-control-rescue:CONN_6-capteur-rescue -> remote-control-rescue:CONN_6-capteur-rescue-remote-control-rescue
- P2, P3: symbol remote-control-rescue:CONN_4-capteur-rescue -> remote-control-rescue:CONN_4-capteur-rescue-remote-control-rescue
- R1: symbol Device:R_Small -> remote-control-rescue:R_Small-Device
- R2: symbol remote-control-rescue:R-RESCUE-capteur-capteur-rescue -> remote-control-rescue:R-RESCUE-capteur-capteur-rescue-remote-control-rescue
- TVS1: symbol Diode:1.5KExxA -> remote-control-rescue:1.5KExxA-Diode
- U1: symbol remote-control-rescue:PIC18F2xK80-capteur-rescue -> remote-control-rescue:PIC18F2xK80-capteur-rescue-remote-control-rescue
- U2: symbol remote-control-rescue:MCP2562-capteur-rescue -> remote-control-rescue:MCP2562-capteur-rescue-remote-control-rescue
- U3: symbol remote-control-rescue:ZPT-RFsol -> remote-control-rescue:ZPT-RFsol-remote-control-rescue
- U4: symbol remote-control-rescue:uA78M33-capteur-rescue -> remote-control-rescue:uA78M33-capteur-rescue-remote-control-rescue
- U5: symbol remote-control-rescue:uA78M05-capteur-rescue -> remote-control-rescue:uA78M05-capteur-rescue-remote-control-rescue
- Y1: symbol Device:Crystal_Small -> remote-control-rescue:Crystal_Small-Device
Changed lines of the file:
@@
 EESchema Schematic File Version 4
-LIBS:remote-control-cache
-EELAYER 29 0
+EELAYER 30 0
 EELAYER END
 $Descr A4 11693 8268
@@
 $EndDescr
 $Comp
-L remote-control-rescue:MCP2562-capteur-rescue U2
+L remote-control-rescue:MCP2562-capteur-rescue-remote-control-rescue U2
 U 1 1 5D07804E
 P 6700 2250
@@
 $EndComp
 $Comp
-L remote-control-rescue:PIC18F2xK80-capteur-rescue U1
+L remote-control-rescue:PIC18F2xK80-capteur-rescue-remote-control-rescue U1
 U 1 1 5D07804F
 P 5350 5450
@@
 $EndComp
 $Comp
-L remote-control-rescue:uA78M33-capteur-rescue U4
+L remote-control-rescue:uA78M33-capteur-rescue-remote-control-rescue U4
 U 1 1 5D078050
 P 8950 4900
@@
 $EndComp
 $Comp
-L remote-control-rescue:GND-RESCUE-capteur-capteur-rescue #PWR014
+L remote-control-rescue:GND-RESCUE-capteur-capteur-rescue-remote-control-rescue #PWR014
 U 1 1 5D078051
 P 9350 4900
@@
 $EndComp
 $Comp
-L power:+12V #PWR012
+L remote-control-rescue:+12V-power #PWR012
 U 1 1 5D078052
 P 8900 4400
@@
 $EndComp
 $Comp
-L remote-control-rescue:+3.3V-RESCUE-capteur-capteur-rescue #PWR013
+L remote-control-rescue:+3.3V-RESCUE-capteur-capteur-rescue-remote-control-rescue #PWR013
 U 1 1 5D078053
 P 8900 5600
@@
 $EndComp
 $Comp
-L remote-control-rescue:C-RESCUE-capteur-capteur-rescue C4
+L remote-control-rescue:C-RESCUE-capteur-capteur-rescue-remote-control-rescue C4
 U 1 1 5D078054
 P 5250 6700
@@
 $EndComp
 $Comp
-L remote-control-rescue:+3.3V-RESCUE-capteur-capteur-rescue #PWR08
+L remote-control-rescue:+3.3V-RESCUE-capteur-capteur-rescue-remote-control-rescue #PWR08
 U 1 1 5D078048
 P 6900 5450
@@
 $EndComp
 $Comp
-L remote-control-rescue:+3.3V-RESCUE-capteur-capteur-rescue #PWR09
+L remote-control-rescue:+3.3V-RESCUE-capteur-capteur-rescue-remote-control-rescue #PWR09
 U 1 1 5D078056
 P 7350 2550
@@
 $EndComp
 $Comp
-L remote-control-rescue:GND-RESCUE-capteur-capteur-rescue #PWR02
+L remote-control-rescue:GND-RESCUE-capteur-capteur-rescue-remote-control-rescue #PWR02
 U 1 1 5D078057
 P 4950 6750
@@
 $EndComp
 $Comp
-L remote-control-rescue:GND-RESCUE-capteur-capteur-rescue #PWR04
+L remote-control-rescue:GND-RESCUE-capteur-capteur-rescue-remote-control-rescue #PWR04
 U 1 1 5D078058
 P 6700 3000
@@
 $EndComp
 $Comp
-L power:+5V #PWR03
+L remote-control-rescue:+5V-power #PWR03
 U 1 1 5D078059
 P 6700 1550
@@
 $EndComp
 $Comp
-L Device:C_Small C6
+L remote-control-rescue:C_Small-Device-remote-control-rescue C6
 U 1 1 5D07805A
 P 7200 2750
@@
 $EndComp
 $Comp
-L remote-control-rescue:GND-RESCUE-capteur-capteur-rescue #PWR07
+L remote-control-rescue:GND-RESCUE-capteur-capteur-rescue-remote-control-rescue #PWR07
 U 1 1 5D07805C
 P 6900 5150
@@
 PGD
 $Comp
-L power:PWR_FLAG #PWR_PIC01
+L remote-control-rescue:PWR_FLAG-power #PWR_PIC01
 U 1 1 5D07805D
 P 6850 6350
@@
 $EndComp
 $Comp
-L remote-control-rescue:CP1-RESCUE-capteur-capteur-rescue C8
+L remote-control-rescue:CP1-RESCUE-capteur-capteur-rescue-remote-control-rescue C8
 U 1 1 5D07805F
 P 9100 5450
@@
 $EndComp
 $Comp
-L remote-control-rescue:CP1-RESCUE-capteur-capteur-rescue C2
+L remote-control-rescue:CP1-RESCUE-capteur-capteur-rescue-remote-control-rescue C2
 U 1 1 5D078060
 P 4700 6700
@@
 $EndComp
 $Comp
-L remote-control-rescue:CONN_6-capteur-rescue P1
+L remote-control-rescue:CONN_6-capteur-rescue-remote-control-rescue P1
 U 1 1 00000000
 P 7350 5300
@@
 NoConn ~ 5450 4450
 $Comp
-L remote-control-rescue:uA78M05-capteur-rescue U5
+L remote-control-rescue:uA78M05-capteur-rescue-remote-control-rescue U5
 U 1 1 5D078038
 P 9800 4900
@@
 $EndComp
 $Comp
-L remote-control-rescue:GND-RESCUE-capteur-capteur-rescue #PWR017
+L remote-control-rescue:GND-RESCUE-capteur-capteur-rescue-remote-control-rescue #PWR017
 U 1 1 5D078039
 P 10200 4900
@@
 $EndComp
 $Comp
-L power:+12V #PWR015
+L remote-control-rescue:+12V-power #PWR015
 U 1 1 5D07803A
 P 9750 4400
@@
 $EndComp
 $Comp
-L remote-control-rescue:CP1-RESCUE-capteur-capteur-rescue C9
+L remote-control-rescue:CP1-RESCUE-capteur-capteur-rescue-remote-control-rescue C9
 U 1 1 5D07802E
 P 9950 5450
@@
 $EndComp
 $Comp
-L power:+5V #PWR016
+L remote-control-rescue:+5V-power #PWR016
 U 1 1 5D07803C
 P 9750 5600
@@
 	8900 4400 8900 4500
 $Comp
-L remote-control-rescue:R-RESCUE-capteur-capteur-rescue R2
+L remote-control-rescue:R-RESCUE-capteur-capteur-rescue-remote-control-rescue R2
 U 1 1 5D078047
 P 7550 5200
@@
 	7000 5150 7550 5150
 $Comp
-L Device:Crystal_Small Y1
+L remote-control-rescue:Crystal_Small-Device Y1
 U 1 1 5D0873A6
 P 4800 4300
@@
 $EndComp
 $Comp
-L remote-control-rescue:C_Small-Device C1
+L remote-control-rescue:C_Small-Device-remote-control-rescue C1
 U 1 1 5D089370
 P 4700 4000
@@
 $EndComp
 $Comp
-L remote-control-rescue:C_Small-Device C3
+L remote-control-rescue:C_Small-Device-remote-control-rescue C3
 U 1 1 5D0896AC
 P 4900 4000
@@
 $EndComp
 $Comp
-L remote-control-rescue:GND-RESCUE-capteur-capteur-rescue #PWR01
+L remote-control-rescue:GND-RESCUE-capteur-capteur-rescue-remote-control-rescue #PWR01
 U 1 1 5D08A8C6
 P 4800 3800
@@
 NoConn ~ 4450 4450
 $Comp
-L remote-control-rescue:ZPT-RFsol U3
+L remote-control-rescue:ZPT-RFsol-remote-control-rescue U3
 U 1 1 5D06B913
 P 7750 3750
@@
 $EndComp
 $Comp
-L remote-control-rescue:C-RESCUE-capteur-capteur-rescue C5
+L remote-control-rescue:C-RESCUE-capteur-capteur-rescue-remote-control-rescue C5
 U 1 1 5D06C1C4
 P 6800 3700
@@
 	7000 3900 6800 3900
 $Comp
-L remote-control-rescue:GND-RESCUE-capteur-capteur-rescue #PWR06
+L remote-control-rescue:GND-RESCUE-capteur-capteur-rescue-remote-control-rescue #PWR06
 U 1 1 5D0711B2
 P 6800 3400
@@
 Connection ~ 6800 3500
 $Comp
-L remote-control-rescue:+3.3V-RESCUE-capteur-capteur-rescue #PWR05
+L remote-control-rescue:+3.3V-RESCUE-capteur-capteur-rescue-remote-control-rescue #PWR05
 U 1 1 5D0739C8
 P 6750 3900
@@
 	5650 4200 5650 4450
 $Comp
-L Device:R_Small R1
+L remote-control-rescue:R_Small-Device R1
 U 1 1 5D06D0F4
 P 7150 4000
@@
 $EndComp
 $Comp
-L Device:LED D1
+L remote-control-rescue:LED-Device D1
 U 1 1 5D0700DD
 P 6950 4100
@@
 	7150 4100 7100 4100
 $Comp
-L Connector:Conn_Coaxial J1
+L remote-control-rescue:Conn_Coaxial-Connector J1
 U 1 1 5D0839F1
 P 7200 3250
@@
 	8450 1850 9200 1850
 $Comp
-L power:PWR_FLAG #U01
+L remote-control-rescue:PWR_FLAG-power #U01
 U 1 1 5D07803E
 P 7550 1450
@@
 $EndComp
 $Comp
-L Device:D_Schottky_Small D2
+L remote-control-rescue:D_Schottky_Small-Device D2
 U 1 1 5D07803D
 P 7850 1550
@@
 $EndComp
 $Comp
-L remote-control-rescue:CP1-RESCUE-capteur-capteur-rescue C7
+L remote-control-rescue:CP1-RESCUE-capteur-capteur-rescue-remote-control-rescue C7
 U 1 1 5D07805E
 P 7550 1750
@@
 $EndComp
 $Comp
-L power:+12V #PWR011
+L remote-control-rescue:+12V-power #PWR011
 U 1 1 5D07804D
 P 7450 1550
@@
 $EndComp
 $Comp
-L remote-control-rescue:GND-RESCUE-capteur-capteur-rescue #PWR010
+L remote-control-rescue:GND-RESCUE-capteur-capteur-rescue-remote-control-rescue #PWR010
 U 1 1 5D07804C
 P 7400 1950
@@
 $EndComp
 $Comp
-L power:PWR_FLAG #U02
+L remote-control-rescue:PWR_FLAG-power #U02
 U 1 1 5D07804B
 P 8450 1450
@@
 $EndComp
 $Comp
-L power:PWR_FLAG #GND01
+L remote-control-rescue:PWR_FLAG-power #GND01
 U 1 1 5D07804A
 P 8150 1450
@@
 12Vin
 $Comp
-L remote-control-rescue:CONN_4-capteur-rescue P2
+L remote-control-rescue:CONN_4-capteur-rescue-remote-control-rescue P2
 U 1 1 5D078049
 P 8800 2000
@@
 $EndComp
 $Comp
-L remote-control-rescue:CONN_4-capteur-rescue P3
+L remote-control-rescue:CONN_4-capteur-rescue-remote-control-rescue P3
 U 1 1 5D078055
 P 9550 2000
@@
 	4150 5050 7000 5050
 $Comp
-L Diode:1.5KExxA TVS1
+L remote-control-rescue:1.5KExxA-Diode TVS1
 U 1 1 5D0EC305
 P 8250 1750
